File: sd-rom-design/sd-rom.kicad_pcb (KiCad board)
At the start: 2 copper layers, 157.8 x 100 mm, 12 parts, among them J1 JAE50, J2 Conn_01x40, J3 Conn_01x40, J4 SD44, J5 Conn_01x04_Male, U1 ATtiny13A-SSU, U2 AMS1117-3.3

Commit message: board variant 3
Parts:
- moved J1 105.1 mm to (39.8, 38.3), turned to 225 degrees
- moved U2 96.0 mm to (91.8, 16.4), turned to 0 degrees
- moved R2 93.1 mm to (40.1, 57.2), turned to 135 degrees
- moved J2 84.9 mm to (56.1, 59.3), turned to 225 degrees
- moved C1 84.8 mm to (83.8, 16.4), turned to 90 degrees
- moved R1 78.7 mm to (77.8, 9.40), turned to 0 degrees
- moved U1 76.4 mm to (77.8, 16.4), turned to 90 degrees
- moved R3 75.3 mm to (77.8, 23.4), turned to 0 degrees
- moved C2 68.1 mm to (71.8, 16.4), turned to 270 degrees
- moved J5 11.1 mm to (16.3, 70.2), turned to 90 degrees
- moved J4 5.39 mm to (56.0, 86.2)
Other:
- board size 157.8 x 100 mm -> 90.1 x 100 mm

Commit message: parts found in local shop
Parts:
- J4: footprint sd-rom:PinHeader_2x22_P2.00mm_Horizontal -> sd-rom:PinSocket_2x22_P2.00mm_Horizontal
- moved J4 41.9 mm to (84.7, 55.7), turned to 315 degrees

Commit message: tracing in progress
Parts:
- moved R2 9.68 mm to (47.7, 51.2), turned to 45 degrees
- moved J4 4.27 mm to (81.6, 52.8)
Routing:
- net GNDREF: track 0.00 -> 135.7 mm, vias 1 -> 5
- net GND: track 0.00 -> 105.1 mm, vias 0 -> 1
- net Net-(J5-Pad1): track 0.00 -> 98.8 mm, vias 0 -> 1
- net /Button: track 0.00 -> 96.6 mm
- net Net-(J5-Pad3): track 0.00 -> 95.7 mm
- net Net-(J1-Pad47): track 0.00 -> 37.3 mm
- net Net-(J1-Pad38): track 0.00 -> 36.0 mm
- net Net-(J1-Pad28): track 0.00 -> 33.9 mm, vias 0 -> 2
- net Net-(J1-Pad30): track 0.00 -> 33.8 mm, vias 0 -> 2
- net Net-(J1-Pad32): track 0.00 -> 33.8 mm, vias 0 -> 2
- net Net-(J1-Pad24): track 0.00 -> 33.5 mm, vias 0 -> 2
- net Net-(J1-Pad34): track 0.00 -> 33.5 mm, vias 0 -> 2
- net Net-(J1-Pad22): track 0.00 -> 33.4 mm, vias 0 -> 2
- net Net-(J1-Pad36): track 0.00 -> 33.2 mm, vias 0 -> 2
- net Net-(C2-Pad1): track 0.00 -> 32.1 mm
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
Commit message: pcb design finished
Parts:
- moved J4 1.89 mm to (83.4, 52.3)
Routing:
- net GND: track 105.1 -> 300.6 mm, vias 1 -> 2
- net /LedIn: track 4.28 -> 90.7 mm, vias 1 -> 2
- net VCC: track 5.38 -> 88.3 mm, vias 0 -> 2
- net Net-(J3-Pad40): track 0.00 -> 41.9 mm
- net Net-(J3-Pad37): track 0.00 -> 38.3 mm, vias 0 -> 1
- net Net-(J3-Pad38): track 0.00 -> 36.9 mm
- net Net-(J3-Pad35): track 0.00 -> 36.1 mm, vias 0 -> 1
- net Net-(J3-Pad36): track 0.00 -> 34.8 mm
- net Net-(J3-Pad33): track 0.00 -> 34.4 mm, vias 0 -> 1
- net Net-(J3-Pad31): track 0.00 -> 33.1 mm, vias 0 -> 1
- net Net-(J3-Pad34): track 0.00 -> 32.4 mm
- net Net-(J3-Pad29): track 0.00 -> 31.9 mm, vias 0 -> 1
- net Net-(J3-Pad32): track 0.00 -> 31.3 mm
- net Net-(J3-Pad27): track 0.00 -> 30.7 mm, vias 0 -> 1
- net Net-(J3-Pad25): track 0.00 -> 29.4 mm
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Other:
- rule trace_min: 0.2 -> 0.153
- rule via_min_size: 0.4 -> 0.153
